File: Pocket386.kicad_pcb (KiCad board)
At the start: 2 copper layers, 65.6 x 41.4 mm, 19 parts, among them J1 Conn_02x40_Odd_Even, U1 Pico, U2 SN74CB3T3257, U3 SN74CB3T3257, U4 74AHC14, U5 74LVC00, U6 SN74CB3T3245, U7 APS6404L-3SQN-SN, U8 74LVC1G00, U9 74LVC1G06

Commit message: Add back [final?] signals?
Parts:
- added D1: 1A 20V Schottky, Diode_SMD:D_SOD-123, B.Cu at (173.1, 111.0)
- added JP2: USB Power, Connector_PinHeader_2.54mm:PinHeader_1x02_P2.54mm_Vertical, F.Cu at (162.8, 116.7)
Connections:
- J1 pad 45: IORDY -> I/OCHRDY
- U1 pad 1: unconnected-(U1-GPIO0-Pad1) -> SPI_RX
- U1 pad 10: unconnected-(U1-GPIO7-Pad10) -> AD1
- U1 pad 11: unconnected-(U1-GPIO8-Pad11) -> AD2
- U1 pad 12: unconnected-(U1-GPIO9-Pad12) -> AD3
- U1 pad 13: unconnected-(U1-GND-Pad13) -> GND
- U1 pad 14: unconnected-(U1-GPIO10-Pad14) -> AD4
- U1 pad 15: unconnected-(U1-GPIO11-Pad15) -> AD5
- U1 pad 16: unconnected-(U1-GPIO12-Pad16) -> AD6
- U1 pad 17: unconnected-(U1-GPIO13-Pad17) -> AD7
- U1 pad 18: unconnected-(U1-GND-Pad18) -> GND
- U1 pad 19: unconnected-(U1-GPIO14-Pad19) -> RA8
- U1 pad 2: unconnected-(U1-GPIO1-Pad2) -> ~{SPI_CS}
- U1 pad 20: unconnected-(U1-GPIO15-Pad20) -> RA9
- U1 pad 21: unconnected-(U1-GPIO16-Pad21) -> DIN
- U1 pad 22: unconnected-(U1-GPIO17-Pad22) -> BCK
- U1 pad 23: unconnected-(U1-GND-Pad23) -> GND
- U1 pad 24: unconnected-(U1-GPIO18-Pad24) -> LRCK
- U1 pad 25: unconnected-(U1-GPIO19-Pad25) -> ~{RDACK}
- U1 pad 26: unconnected-(U1-GPIO20-Pad26) -> RTC
- U1 pad 27: unconnected-(U1-GPIO21-Pad27) -> RIRQ
- U1 pad 28: unconnected-(U1-GND-Pad28) -> GND
- U1 pad 29: unconnected-(U1-GPIO22-Pad29) -> RDRQ
- U1 pad 3: unconnected-(U1-GND-Pad3) -> GND
- U1 pad 30: unconnected-(U1-RUN-Pad30) -> RUN
- U1 pad 31: unconnected-(U1-GPIO26_ADC0-Pad31) -> ~{RI/OCHRDY}
- U1 pad 32: unconnected-(U1-GPIO27_ADC1-Pad32) -> ADS
- U1 pad 33: unconnected-(U1-AGND-Pad33) -> GND
- U1 pad 34: unconnected-(U1-GPIO28_ADC2-Pad34) -> UART_TX
- U1 pad 36: unconnected-(U1-3V3-Pad36) -> +3.3V
- U1 pad 38: unconnected-(U1-GND-Pad38) -> GND
- U1 pad 39: unconnected-(U1-VSYS-Pad39) -> /VSYS
- U1 pad 4: unconnected-(U1-GPIO2-Pad4) -> SPI_SCK
- U1 pad 40: unconnected-(U1-VBUS-Pad40) -> Net-(JP2-A)
- U1 pad 42: unconnected-(U1-GND-Pad42) -> GND
- U1 pad 5: unconnected-(U1-GPIO3-Pad5) -> SPI_TX
- U1 pad 6: unconnected-(U1-GPIO4-Pad6) -> ~{RIOW}
- U1 pad 7: unconnected-(U1-GPIO5-Pad7) -> ~{RIOR}
- U1 pad 8: unconnected-(U1-GND-Pad8) -> GND
- U1 pad 9: unconnected-(U1-GPIO6-Pad9) -> AD0
Routing:
- added copper zone on B.Cu, net GND
- added copper zone on F.Cu, net GND
